File: reaction-wheel-bldc-motor-control-pcb.kicad_sch (KiCad schematic)
At the start: 34 parts, among them J1 USB_C_Receptacle_USB2.0_16P, J7 Conn_01x04_Pin, J8 Conn_01x04_Pin, SW1 SW_SPDT, SW3 SW_SPST, U1 STM32G431CBUx, U2 AS5047D, U3 DRV8311H, U5 USBLC6-2SC6, U7 TJA1051T-3, Y1 16MHz

Commit message: schematic almost complete
Parts:
- removed C25, C26: 100n, Capacitor_SMD:C_0805_2012Metric_Pad1.18x1.45mm_HandSolder, symbol Device:C_Small
- removed D3: NUP2105L, Package_TO_SOT_SMD:SOT-23, symbol Power_Protection:NUP2105L
- removed R2: 10k, Resistor_SMD:R_0402_1005Metric, symbol Device:R
- removed SW1: SW_SPDT, Button_Switch_THT:SW_E-Switch_EG1224_SPDT_Angled, symbol Switch:SW_SPDT
- removed U7: TJA1051T-3, Package_SO:SOIC-8_3.9x4.9mm_P1.27mm, symbol Interface_CAN_LIN:TJA1051T-3
- added C27: 1u, Capacitor_SMD:C_0805_2012Metric_Pad1.18x1.45mm_HandSolder, symbol Device:C_Small
- added C28, C31, C33, C35: 0.1u, Capacitor_SMD:C_0805_2012Metric_Pad1.18x1.45mm_HandSolder, symbol Device:C_Small
- added C29: 4.7u, Capacitor_SMD:C_0805_2012Metric_Pad1.18x1.45mm_HandSolder, symbol Device:C_Small
- added C30: 100n, Capacitor_SMD:C_0805_2012Metric_Pad1.18x1.45mm_HandSolder, symbol Device:C_Small
- added C32: 22u, Capacitor_SMD:C_0805_2012Metric_Pad1.18x1.45mm_HandSolder, symbol Device:C_Small
- added C34: 10u, Capacitor_SMD:C_0805_2012Metric_Pad1.18x1.45mm_HandSolder, symbol Device:C_Small
- added D1, D2: SS34, Diode_SMD:D_SMA, symbol Diode:SS34
- added D4: NUP2105L, Package_TO_SOT_SMD:SOT-23, symbol Power_Protection:NUP2105L
- added J2: Conn_01x05_Pin, symbol Connector:Conn_01x05_Pin
- added L1: 2.2u, symbol Device:L
- added R1, R4: 100k, symbol Device:R
- added R3: 30.1K, symbol Device:R
- added R5: 10K, symbol Device:R
- added U4: SN65HVD231, Package_SO:SOIC-8_3.9x4.9mm_P1.27mm, symbol Interface_CAN_LIN:SN65HVD231
- added U6: TPS562200, Package_TO_SOT_SMD:SOT-23-6, symbol Regulator_Switching:TPS562200
Connections:
- net +3.3V: now also J7.1 (Pin_1), J8.1 (Pin_1), U2.11 (VDD), U2.12 (VDD3V3), U3.18 (INLA), U3.19 (INLB), U3.20 (INLC), C27.2, C32.2, J2.1 (Pin_1), L1.2, R1.1, R4.2, R5.2, U4.3 (VCC)
- net +3.3VA: now also U1.20 (VREF+)
- net CAN_H: now also D4.2 (K), U4.7 (CANH)
- net CAN_L: now also D4.1 (K), U4.6 (CANL)
- net CAN_RX: now also U4.4 (R)
- net CAN_TX: now also U4.1 (D)
- net GND: now also U1.49 (VSS), U2.13 (GND), U2.5 (TST), U3.16 (AGND), U3.25 (PGND), U3.9 (PGND), C27.1, C28.2, C29.2, C30.1, C32.1, C33.1, C34.1, D4.3 (A), J2.5 (Pin_5), R3.2, U4.2 (GND), U4.8 (Rs), U6.1 (GND)
- net SPI1_CS: now reaches U2.1 (~{CS})
- net SPI1_CS: now also U1.12 (PA4)
- net SPI1_SCK: now reaches U2.2 (CLK)
- net SPI1_SCK: now also U1.13 (PA5)
- net SPI1_MISO: now reaches U2.3 (MISO)
- net SPI1_MISO: now also U1.14 (PA6)
- net SPI1_MOSI: now reaches U2.4 (MOSI)
- net SPI1_MOSI: now also U1.15 (PA7)
- net FAULT: now reaches U3.1 (~{FAULT})
- net FAULT: now also U1.25 (PB12), R5.1
- net MOTOR_C: now reaches U3.10 (OUTA)
- net MOTOR_C: now also J2.4 (Pin_4)
- net MOTOR_B: now reaches U3.11 (OUTB)
- net MOTOR_B: now also J2.3 (Pin_3)
- net MOTOR_A: now reaches U3.12 (OUTC)
- net MOTOR_A: now also J2.2 (Pin_2)
- net PA10: now reaches U3.13 (INHC)
- net PA10: now also U1.32 (PA10)
- net PA9: now reaches U3.14 (INHB)
- net PA9: now also U1.31 (PA9)
- net PA8: now reaches U3.15 (INHA)
- net PA8: now also U1.30 (PA8)
- net at U3.17 (AVDD): now also C29.1
- net at U3.2 (CSAREF): now also C28.1
- net SLEEP: now reaches U3.24 (~{SLEEP})
- net SLEEP: now also U1.26 (PB13), R4.1
- net PA0: now reaches U3.3 (SOC)
- net PA0: now also U1.8 (PA0)
- net PA1: now reaches U3.4 (SOB)
- net PA1: now also U1.9 (PA1)
- net PB0: now reaches U3.5 (SOA)
- net PB0: now also U1.17 (PB0)
- net at U3.6 (CP): now also C35.1
- net VBAT: now reaches U3.7 (VIN_AVDD)
- net VBAT: now also U3.8 (VM), C33.2, C34.2, C35.2, D2.2 (A)
- net VBUS renamed +5V
- net +5V: now also D1.2 (A); no longer J7.1 (Pin_1), J8.1 (Pin_1)
- new net: D1.1 (K), D2.1 (K), U6.3 (VIN), U6.5 (EN)
- new net: R1.2, R3.1, U6.4 (VFB)
- new net: C31.2, L1.1, U6.2 (SW)
- new net: C31.1, U6.6 (VBST)
- new net: C30.2, U4.5 (Vref)
- no-connect marks 2 -> 29
Other:
- note added: "3.3V Buck Regulator"
- note added: "Encoder"
- note added: "Motor Driver"
- note added: "Motor Headers"
- note added: "Mounting Holes"
- note added: "Power Flags"
- note added: "Reset Switch"
- note removed: "Reset and Boot Switches"
- moved on the sheet: C12, C13, C14, H1, H2, H3, H4, J1, J7, J8, R13, R14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

Commit message: started with pcb routing
Parts:
- removed J2: Conn_01x05_Pin, symbol Connector:Conn_01x05_Pin
- added J3: Conn_01x03_Pin, Connector_PinHeader_2.54mm:PinHeader_1x03_P2.54mm_Vertical, symbol Connector:Conn_01x03_Pin
- added J5: Conn_01x04_Pin, Connector_PinHeader_2.54mm:PinHeader_1x04_P2.54mm_Vertical, symbol Connector:Conn_01x04_Pin
- added J6: Conn_01x06_Pin, Connector_PinHeader_2.54mm:PinHeader_1x06_P2.54mm_Vertical, symbol Connector:Conn_01x06_Pin
- added MT1: Screw_Terminal, TerminalBlock_Phoenix:TerminalBlock_Phoenix_MKDS-1,5-2-5.08_1x02_P5.08mm_Horizontal, symbol Connector:Screw_Terminal_01x02
- C13: renamed from C27; footprint Capacitor_SMD:C_0805_2012Metric_Pad1.18x1.45mm_HandSolder -> Capacitor_SMD:C_0603_1608Metric
- C14: renamed from C28; footprint Capacitor_SMD:C_0805_2012Metric_Pad1.18x1.45mm_HandSolder -> Capacitor_SMD:C_0402_1005Metric
- C15: renamed from C33; footprint Capacitor_SMD:C_0805_2012Metric_Pad1.18x1.45mm_HandSolder -> Capacitor_SMD:C_0402_1005Metric
- C16: renamed from C34; footprint Capacitor_SMD:C_0805_2012Metric_Pad1.18x1.45mm_HandSolder -> Capacitor_SMD:C_0603_1608Metric
- C17: renamed from C29; footprint Capacitor_SMD:C_0805_2012Metric_Pad1.18x1.45mm_HandSolder -> Capacitor_SMD:C_0603_1608Metric
- C18: renamed from C35; footprint Capacitor_SMD:C_0805_2012Metric_Pad1.18x1.45mm_HandSolder -> Capacitor_SMD:C_0402_1005Metric
- C19: renamed from C30; footprint Capacitor_SMD:C_0805_2012Metric_Pad1.18x1.45mm_HandSolder -> Capacitor_SMD:C_0402_1005Metric
- C20: renamed from C31; footprint Capacitor_SMD:C_0805_2012Metric_Pad1.18x1.45mm_HandSolder -> Capacitor_SMD:C_0402_1005Metric
- C21: renamed from C32; footprint Capacitor_SMD:C_0805_2012Metric_Pad1.18x1.45mm_HandSolder -> Capacitor_SMD:C_0603_1608Metric
- J4: renamed from J1; footprint (none) -> Connector_USB:USB_C_Receptacle_G-Switch_GT-USB-7010ASV
- L1: footprint (none) -> Inductor_SMD:L_0402_1005Metric
- R1: renamed from R13; footprint Resistor_SMD:R_0805_2012Metric_Pad1.20x1.40mm_HandSolder -> Resistor_SMD:R_0402_1005Metric
- R2: renamed from R14; footprint Resistor_SMD:R_0805_2012Metric_Pad1.20x1.40mm_HandSolder -> Resistor_SMD:R_0402_1005Metric
- R3: renamed from R5; footprint (none) -> Resistor_SMD:R_0402_1005Metric
- R4: footprint (none) -> Resistor_SMD:R_0603_1608Metric
- R5: renamed from R1; footprint (none) -> Resistor_SMD:R_0603_1608Metric
- R6: renamed from R3; footprint (none) -> Resistor_SMD:R_0603_1608Metric
- SW1: renamed from SW3; footprint (none) -> Button_Switch_SMD:SW_SPST_SKQG_WithStem
- renumbered C3 to C1, C14 to C10, C10 to C11, C7 to C12, C8 to C2, C13 to C3, C11 to C5, C12 to C6, C9 to C7, C5 to C8, C6 to C9, D2 to D1, D1 to D2, D4 to D3, J7 to J1, J8 to J2, U5 to U1, U1 to U2, U2 to U3, U3 to U4, U4 to U5
Connections:
- net +3.3V: now also J5.1 (Pin_1), J6.1 (Pin_1)
- net GND: now also J5.4 (Pin_4), J6.6 (Pin_6), MT1.2 (Pin_2)
- net MOTOR_A: now also J3.1 (Pin_1)
- net MOTOR_B: now also J3.2 (Pin_2)
- net MOTOR_C: now also J3.3 (Pin_3)
- net SPI1_CS: now also J6.5 (Pin_5)
- net SPI1_MISO: now also J6.3 (Pin_3)
- net SPI1_MOSI: now also J6.2 (Pin_2)
- net SPI1_SCK: now also J6.4 (Pin_4)
- net VBAT: now also MT1.1 (Pin_1)
- net I2C1_SCL: now reaches U2.38 (PA15)
- net I2C1_SCL: now also J5.2 (Pin_2)
- net I2C1_SDA: now reaches U2.45 (PB7)
- net I2C1_SDA: now also J5.3 (Pin_3)
- no-connect marks 29 -> 27
Other:
- note added: "Battery Screw Terminal"
- note added: "I2C1 Headers"
- note added: "SPI1 Headers"

Commit message: started with pcb routing
Parts:
- removed C6: 0.1u, Capacitor_SMD:C_0402_1005Metric, symbol Device:C
Changed lines of the file:
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@@
 	)
 	(junction
-		(at 30.48 74.93)
-		(diameter 0)
-		(color 0 0 0 0)
-	)
-	(junction
 		(at 31.75 22.86)
 		(diameter 0)
@@
 	)
 	(junction
-		(at 38.1 74.93)
-		(diameter 0)
-		(color 0 0 0 0)
-	)
-	(junction
 		(at 24.13 44.45)
 		(diameter 0)
@@
 					(unit 1)
 				)
-			)
-		)
-	)
-	(symbol
-		(lib_id "Device:C")
-		(at 34.29 74.93 90)
-		(unit 1)
-		(body_style 1)
-		(exclude_from_sim no)
-		(in_bom yes)
-		(on_board yes)
-		(in_pos_files yes)
-		(dnp no)
-		(property "Reference" "C6"
-			(at 37.846 72.898 90)
-			(show_name no)
-			(do_not_autoplace no)
-			(effects
-				(font
-					(size 1.27 1.27)
-				)
-			)
-		)
-		(property "Value" "0.1u"
-			(at 34.798 78.74 90)
-			(show_name no)
-			(do_not_autoplace no)
-			(effects
-				(font
-					(size 1.27 1.27)
-				)
-			)
-		)
-		(property "Footprint" "Capacitor_SMD:C_0402_1005Metric"
-			(at 38.1 73.9648 0)
-			(hide yes)
-			(show_name no)
-			(do_not_autoplace no)
-			(effects
-				(font
-					(size 1.27 1.27)
-				)
-			)
-		)
-		(property "Datasheet" ""
-			(at 34.29 74.93 0)
-			(hide yes)
-			(show_name no)
-			(do_not_autoplace no)
-			(effects
-				(font
-					(size 1.27 1.27)
-				)
-			)
-		)
-		(property "Description" "Unpolarized capacitor"
-			(at 34.29 74.93 0)
-			(hide yes)
-			(show_name no)
-			(do_not_autoplace no)
-			(effects
-				(font
-					(size 1.27 1.27)
-				)
-			)
-		)
-		(pin "1"
-		)
-		(pin "2"
-		)
-		(instances
-			(project "reaction-wheel-bldc-motor-control-pcb"
-				(path "/c5096c1b-e27c-4190-9cf1-fa68461b3db0"
-					(reference "C6")
-					(unit 1)
-				)

Commit message: routing almost finished
Other:
- moved on the sheet: C14, C15, C16, C17, C18, R3, R4, U2, U4
