File: reaction-wheel-bldc-motor-control-pcb.kicad_sch (KiCad schematic)
At the start: 50 parts, among them J1 Conn_01x04_Pin, J2 Conn_01x04_Pin, J3 Conn_01x03_Pin, J4 USB_C_Receptacle_USB2.0_16P, J5 Conn_01x04_Pin, J6 Conn_01x06_Pin, SW1 SW_SPST, U1 USBLC6-2SC6, U2 STM32G431CBUx, U3 AS5047D, U4 DRV8311H, U5 SN65HVD231, U6 TPS562200, Y1 16MHz

Commit message: changed stm32 from u6 to t6
Parts:
- removed U2: STM32G431CBUx, Package_DFN_QFN:QFN-48-1EP_7x7mm_P0.5mm_EP5.6x5.6mm, symbol MCU_ST_STM32G4:STM32G431CBUx
- added U2: STM32G431CBTx, Package_QFP:LQFP-48_7x7mm_P0.5mm, symbol MCU_ST_STM32G4:STM32G431CBTx
- C1: footprint Capacitor_SMD:C_0603_1608Metric -> Capacitor_SMD:C_0805_2012Metric
- C10: renamed from C11; footprint Capacitor_SMD:C_0402_1005Metric -> Capacitor_SMD:C_0805_2012Metric
- C11: renamed from C12; footprint Capacitor_SMD:C_0402_1005Metric -> Capacitor_SMD:C_0805_2012Metric
- C12: renamed from C13; footprint Capacitor_SMD:C_0603_1608Metric -> Capacitor_SMD:C_0805_2012Metric
- C13: renamed from C14; footprint Capacitor_SMD:C_0402_1005Metric -> Capacitor_SMD:C_0805_2012Metric
- C14: renamed from C15; footprint Capacitor_SMD:C_0402_1005Metric -> Capacitor_SMD:C_0805_2012Metric
- C15: renamed from C16; footprint Capacitor_SMD:C_0603_1608Metric -> Capacitor_SMD:C_0805_2012Metric
- C16: renamed from C17; footprint Capacitor_SMD:C_0603_1608Metric -> Capacitor_SMD:C_0805_2012Metric
- C17: renamed from C18; footprint Capacitor_SMD:C_0402_1005Metric -> Capacitor_SMD:C_0805_2012Metric
- C18: renamed from C19; footprint Capacitor_SMD:C_0402_1005Metric -> Capacitor_SMD:C_0805_2012Metric
- C19: renamed from C20; footprint Capacitor_SMD:C_0402_1005Metric -> Capacitor_SMD:C_0805_2012Metric
- C2, C3, C4, C5: footprint Capacitor_SMD:C_0402_1005Metric -> Capacitor_SMD:C_0805_2012Metric
- C20: renamed from C21; footprint Capacitor_SMD:C_0603_1608Metric -> Capacitor_SMD:C_0805_2012Metric
- C6: renamed from C7; footprint Capacitor_SMD:C_0402_1005Metric -> Capacitor_SMD:C_0805_2012Metric
- C7: renamed from C8; footprint Capacitor_SMD:C_0402_1005Metric -> Capacitor_SMD:C_0805_2012Metric
- C8: renamed from C9; footprint Capacitor_SMD:C_0402_1005Metric -> Capacitor_SMD:C_0805_2012Metric
- C9: renamed from C10; footprint Capacitor_SMD:C_0402_1005Metric -> Capacitor_SMD:C_0805_2012Metric
Connections:
- net +3.3V: now also U2.1 (VBAT), U2.24 (VDD), U2.36 (VDD), U2.48 (VDD)
- net +3.3VA: now also U2.20 (VREF+), U2.21 (VDDA)
- net CAN_RX: now also U2.45 (PB8)
- net CAN_TX: now also U2.46 (PB9)
- net FAULT: now also U2.26 (PB12)
- net GND: now also U2.19 (VSSA), U2.23 (VSS), U2.35 (VSS), U2.47 (VSS)
- net HSE_IN: now also U2.5 (PF0)
- net HSE_OUT: now also U2.6 (PF1)
- net I2C1_SCL: now also U2.39 (PA15)
- net I2C1_SDA: now also U2.44 (PB7)
- net NRST: now also U2.7 (PG10)
- net PA0: now also U2.8 (PA0)
- net PA1: now also U2.9 (PA1)
- net PA10: now also U2.32 (PA10)
- net PA8: now also U2.30 (PA8)
- net PA9: now also U2.31 (PA9)
- net PB0: now also U2.16 (PB0)
- net SLEEP: now also U2.27 (PB13)
- net SPI1_CS: now also U2.12 (PA4)
- net SPI1_MISO: now also U2.14 (PA6)
- net SPI1_MOSI: now also U2.15 (PA7)
- net SPI1_SCK: now also U2.13 (PA5)
- net SWDCLK: now also U2.38 (PA14)
- net SWDIO: now also U2.37 (PA13)
- net USB_D+: now also U2.34 (PA12)
- net USB_D-: now also U2.33 (PA11)
- no-connect marks 27 -> 23

Commit message: complete drv8311 connections
Parts:
- added R7: 47k, Resistor_SMD:R_0603_1608Metric, symbol Device:R
Connections:
- net +3.3VA: now also U4.23 (MODE)
- net GND: now also R7.1
- net at U4.22 (SLEW): now also R7.2
- no-connect marks 23 -> 24
